File: designs/sepic/pcb/sepic/_restore_backup_2026-09-10T13-58-03-979/sepic.kicad_pcb (KiCad board)
At the start: 2 copper layers, 22 parts, among them J2 output, J3 pwm, Q1 irfz44n, U1 INA240A1D, U2 INA240A1D, U3 TC4422

Commit message: first pcb layout attempt
Parts:
- moved U2 80.6 mm to (196.5, 141.5)
- moved iL1 76.4 mm to (165.4, 145.0), turned to 0 degrees
- moved Vcs1 67.8 mm to (160.8, 145.0), turned to 0 degrees
- moved iL2 61.4 mm to (170.0, 145.0), turned to 0 degrees
- moved Co2 58.4 mm to (194.0, 89.5), turned to 0 degrees
- moved Co1 55.0 mm to (194.0, 83.9), turned to 0 degrees
- moved Co3 52.3 mm to (194.0, 95.0), turned to 0 degrees
- moved J2 36.2 mm to (170.7, 108.0), turned to 90 degrees
- moved U3 31.2 mm to (119.4, 142.4)
- moved L1 30.6 mm to (100.0, 77.5)
- moved D1 28.5 mm to (149.4, 77.5), turned to 0 degrees
- moved R_c1 23.3 mm to (115.4, 77.0)
- moved Current_sensor1 23.0 mm to (87.5, 118.0), turned to 0 degrees
- moved U1 22.2 mm to (95.0, 91.0)
- moved R_c2 19.3 mm to (137.5, 124.7), turned to 90 degrees
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