File: designs/sepic/pcb/sepic/sepic.kicad_pcb (KiCad board)
At the start: 2 copper layers, 22 parts, among them J2 output, J3 pwm, Q1 irfz44n, U1 INA240A1D, U2 INA240A1D, U3 TC4422

Commit message: blank
Parts:
- U1, U2: moved to B.Cu
- turned U1 to 180 degrees
- turned U2 to 180 degrees

Commit message: pcb
Parts:
- added C1: 2.2u, Capacitor_THT:C_Disc_D5.0mm_W2.5mm_P2.50mm, F.Cu at (103.2, 118.8)
- R_g1: value 10m -> 10
- moved J2 61.2 mm to (89.3, 91.5), turned to -90 degrees
- moved Current_sensor1 57.9 mm to (146.8, 99.7), turned to 0 degrees
- moved iL2 51.3 mm to (140.0, 88.0)
- moved Q1 46.2 mm to (129.1, 124.5), turned to 180 degrees
- moved Co3 44.6 mm to (99.0, 94.0), turned to -90 degrees
- moved Vcs1 40.2 mm to (139.5, 125.2)
- moved Co1 38.1 mm to (110.0, 94.0), turned to -90 degrees
- moved Co2 37.6 mm to (104.5, 94.0), turned to -90 degrees
- moved U2 31.9 mm to (138.2, 96.0), turned to 0 degrees
- moved R_c2 24.9 mm to (124.7, 105.8)
- moved D1 22.3 mm to (115.4, 94.2), turned to 0 degrees
- moved Cs2 19.5 mm to (128.2, 110.5)
- moved iL1 18.8 mm to (132.8, 88.0)
- moved R_c1 18.1 mm to (113.4, 118.0)
- moved Cs1 18.0 mm to (128.2, 118.0)
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Routing:
- net Net-(Current_sensor1-Pin_2): track 0.00 -> 54.0 mm
- net Net-(Q1-G): track 0.00 -> 28.2 mm
- net Net-(iL1-Pin_2): track 0.00 -> 25.6 mm
- net Net-(J3-Pin_2): track 0.00 -> 20.4 mm
- net /R_cp: track 0.00 -> 20.3 mm
- net /R_cn: track 0.00 -> 14.1 mm
- net /R_c2n: track 0.00 -> 8.00 mm
- net Net-(iL2-Pin_2): track 0.00 -> 6.83 mm
- added copper zone on B.Cu, net /R_c2n
- added copper zone on B.Cu, net /R_cn
- added copper zone on B.Cu, net /R_cp
- added copper zone on B.Cu, net /Vo
- added copper zone on B.Cu, net /pwm
- added copper zone on B.Cu, net GND
- added copper zone on B.Cu, net Net-(D1-A)
- added copper zone on B.Cu, net Net-(input1-Pin_2)
Other:
- board outline added: 68 x 45 mm

Commit message: thinkpad transpport
Parts:
- moved iL1 6.10 mm to (138.8, 89.2)
- moved iL2 5.19 mm to (145.0, 89.2), turned to -90 degrees
- moved D1 0.25 mm to (115.1, 94.2)
Routing:
- net Net-(iL1-Pin_2): track 25.6 -> 32.1 mm
- net Net-(J3-Pin_2): track 20.4 -> 22.6 mm
- net /R_cp: track 20.3 -> 18.1 mm
- net Net-(iL2-Pin_2): track 6.83 -> 5.58 mm
- net (no net): vias 0 -> 4
Other:
- board size 68 x 45 mm -> 76 x 53 mm

Commit message: test
Parts:
- added H1: MountingHole, MountingHole:MountingHole_3.2mm_M3_DIN965, F.Cu at (80.2, 84.2)
- added H2: MountingHole, MountingHole:MountingHole_3.2mm_M3_DIN965, F.Cu at (151.8, 84.0)
- added H3: MountingHole, MountingHole:MountingHole_3.2mm_M3_DIN965, F.Cu at (50.8, 138.5)
- added H4: MountingHole, MountingHole:MountingHole_3.2mm_M3_DIN965, F.Cu at (151.8, 132.5)
Routing:
- net (no net): vias 4 -> 0

Commit message: update
Parts:
- R_c1: footprint Resistor_THT:R_Axial_DIN0207_L6.3mm_D2.5mm_P10.16mm_Horizontal -> Resistor_THT:R_Axial_DIN0414_L11.9mm_D4.5mm_P15.24mm_Horizontal
- R_c2: footprint Resistor_THT:R_Axial_DIN0207_L6.3mm_D2.5mm_P10.16mm_Horizontal -> Resistor_THT:R_Axial_DIN0414_L11.9mm_D4.5mm_P5.08mm_Vertical
- moved R_c2 10.8 mm to (134.0, 100.4), turned to -90 degrees
- moved Cs1 3.91 mm to (131.1, 115.3)
- moved R_c1 0.45 mm to (113.0, 118.1)
Changed lines of the file:
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@@
 		)
 	)
-	(footprint "Resistor_THT:R_Axial_DIN0207_L6.3mm_D2.5mm_P10.16mm_Horizontal"
+	(footprint "Resistor_THT:R_Axial_DIN0414_L11.9mm_D4.5mm_P15.24mm_Horizontal"
 		(layer "F.Cu")
-		(at 113.42 118)
-		(descr "Resistor, Axial_DIN0207 series, Axial, Horizontal, pin pitch=10.16mm, 0.25W = 1/4W, length*diameter=6.3*2.5mm^2, http://cdn-reichelt.de/documents/datenblatt/B400/1_4W%23YAG.pdf")
-		(tags "Resistor Axial_DIN0207 series Axial Horizontal pin pitch 10.16mm 0.25W = 1/4W length 6.3mm diameter 2.5mm")
+		(at 112.98 118.1)
+		(descr "Resistor, Axial_DIN0414 series, Axial, Horizontal, pin pitch=15.24mm, 2W, length*diameter=11.9*4.5mm^2, http://www.vishay.com/docs/20128/wkxwrx.pdf")
+		(tags "Resistor Axial_DIN0414 series Axial Horizontal pin pitch 15.24mm 2W length 11.9mm diameter 4.5mm")
 		(property "Reference" "R_c1"
-			(at 9.08 2.5 0)
+			(at 7.62 -3.37 0)
 			(layer "F.SilkS")
 			(effects
@@
 		)
 		(property "Value" "50m"
-			(at 5.08 2.37 0)
+			(at 7.62 3.37 0)
 			(layer "F.Fab")
 			(effects
@@
 		(duplicate_pad_numbers_are_jumpers no)
 		(fp_line
-			(start 1.04 0)
-			(end 1.81 0)
+			(start 1.44 0)
+			(end 1.55 0)
 			(stroke
 				(width 0.12)
@@
 		)
 		(fp_line
-			(start 9.12 0)
-			(end 8.35 0)
+			(start 13.8 0)
+			(end 13.69 0)
 			(stroke
 				(width 0.12)
@@
 		)
 		(fp_rect
-			(start 1.81 -1.37)
-			(end 8.35 1.37)
+			(start 1.55 -2.37)
+			(end 13.69 2.37)
 			(stroke
 				(width 0.12)
@@
 		)
 		(fp_rect
-			(start -1.05 -1.5)
-			(end 11.21 1.5)
+			(start -1.45 -2.5)
+			(end 16.69 2.5)
 			(stroke
 				(width 0.05)
@@
 		(fp_line
 			(start 0 0)
-			(end 1.93 0)
+			(end 1.67 0)
 			(stroke
 				(width 0.1)
@@
 		)
 		(fp_line
-			(start 10.16 0)
-			(end 8.23 0)
+			(start 15.24 0)
+			(end 13.57 0)
 			(stroke
 				(width 0.1)
@@
 		)
 		(fp_rect
-			(start 1.93 -1.25)
-			(end 8.23 1.25)
+			(start 1.67 -2.25)
+			(end 13.57 2.25)
 			(stroke
 				(width 0.1)
@@
 		)
 		(fp_text user "${REFERENCE}"
-			(at 0 0 0)
+			(at 7.62 0 0)
 			(layer "F.Fab")
 			(effects
@@
 		(pad "1" thru_hole circle
 			(at 0 0)
-			(size 1.6 1.6)
-			(drill 0.8)
+			(size 2.4 2.4)
+			(drill 1.2)
 			(layers "*.Cu" "*.Mask")
 			(remove_unused_layers no)
@@
 		)
 		(pad "2" thru_hole circle
-			(at 10.16 0)
-			(size 1.6 1.6)
-			(drill 0.8)
+			(at 15.24 0)
+			(size 2.4 2.4)
+			(drill 1.2)
 			(layers "*.Cu" "*.Mask")
 			(remove_unused_layers no)
@@
 		)
 		(embedded_fonts no)
-		(model "${KICAD10_3DMODEL_DIR}/Resistor_THT.3dshapes/R_Axial_DIN0207_L6.3mm_D2.5mm_P10.16mm_Horizontal.step"
+		(model "${KICAD10_3DMODEL_DIR}/Resistor_THT.3dshapes/R_Axial_DIN0414_L11.9mm_D4.5mm_P15.24mm_Horizontal.step"
 			(offset
 				(xyz 0 0 0)
@@
 		(pad "" np_thru_hole circle
 			(at 0 0)
-			(size 3.2 3.2)
-			(drill 3.2)
+			(size 2.5 2.5)
+			(drill 2.5)
 			(layers "*.Cu" "*.Mask")
 		)
@@
 		(pad "" np_thru_hole circle
 			(at 0 -0.25)
-			(size 3.2 3.2)
-			(drill 3.2)
+			(size 2.5 2.5)
+			(drill 2.5)
 			(layers "*.Cu" "*.Mask")
 		)
@@
 		(pad "" np_thru_hole circle
 			(at 0 0)
-			(size 3.2 3.2)
-			(drill 3.2)
+			(size 2.5 2.5)
+			(drill 2.5)
 			(layers "*.Cu" "*.Mask")
 		)
@@
 		(pad "" np_thru_hole circle
 			(at 29.5 -6)
-			(size 3.2 3.2)
-			(drill 3.2)
+			(size 2.5 2.5)
+			(drill 2.5)
 			(layers "*.Cu" "*.Mask")
 		)
@@
 		)
 	)
-	(footprint "Resistor_THT:R_Axial_DIN0207_L6.3mm_D2.5mm_P10.16mm_Horizontal"
+	(footprint "Resistor_THT:R_Axial_DIN0414_L11.9mm_D4.5mm_P5.08mm_Vertical"
 		(layer "F.Cu")
-		(at 124.67 105.75)
-		(descr "Resistor, Axial_DIN0207 series, Axial, Horizontal, pin pitch=10.16mm, 0.25W = 1/4W, length*diameter=6.3*2.5mm^2, http://cdn-reichelt.de/documents/datenblatt/B400/1_4W%23YAG.pdf")
-		(tags "Resistor Axial_DIN0207 series Axial Horizontal pin pitch 10.16mm 0.25W = 1/4W length 6.3mm diameter 2.5mm")
+		(at 134 100.37 -90)
+		(descr "Resistor, Axial_DIN0414 series, Axial, Vertical, pin pitch=5.08mm, 2W, length*diameter=11.9*4.5mm^2, http://www.vishay.com/docs/20128/wkxwrx.pdf")
+		(tags "Resistor Axial_DIN0414 series Axial Vertical pin pitch 5.08mm 2W length 11.9mm diameter 4.5mm")
 		(property "Reference" "R_c2"
-			(at 5.08 -2.37 0)
+			(at 2.54 -3.37 90)
 			(layer "F.SilkS")
 			(effects
@@
 		)
 		(property "Value" "50m"
-			(at 1.33 2.5 0)
+			(at 2.54 3.37 90)
 			(layer "F.Fab")
 			(effects
@@
 		)
 		(property "Datasheet" ""
-			(at 0 0 0)
+			(at 0 0 90)
 			(layer "F.Fab")
 			(hide yes)
@@
 		)
 		(property "Description" "Resistor"
-			(at 0 0 0)
+			(at 0 0 90)
 			(layer "F.Fab")
 			(hide yes)
@@
 		(duplicate_pad_numbers_are_jumpers no)
 		(fp_line
-			(start 1.04 0)
-			(end 1.81 0)
-			(stroke
-				(width 0.12)
-				(type solid)
-			)
-			(layer "F.SilkS")
-		)
-		(fp_line
-			(start 9.12 0)
-			(end 8.35 0)
+			(start 2.37 0)
+			(end 3.58 0)
 			(stroke
 				(width 0.12)
@@
 			(layer "F.SilkS")
 		)
-		(fp_rect
-			(start 1.81 -1.37)
-			(end 8.35 1.37)
+		(fp_circle
+			(center 0 0)
+			(end 2.37 0)
 			(stroke
 				(width 0.12)
@@
 		)
 		(fp_rect
-			(start -1.05 -1.5)
-			(end 11.21 1.5)
+			(start -2.5 -2.5)
+			(end 6.53 2.5)
 			(stroke
 				(width 0.05)
@@
 		(fp_line
 			(start 0 0)
-			(end 1.93 0)
+			(end 5.08 0)
 			(stroke
 				(width 0.1)
@@
 			(layer "F.Fab")
 		)
-		(fp_line
-			(start 10.16 0)
-			(end 8.23 0)
-			(stroke
-				(width 0.1)
-				(type solid)
-			)
-			(layer "F.Fab")
-		)
-		(fp_rect
-			(start 1.93 -1.25)
-			(end 8.23 1.25)
+		(fp_circle
+			(center 0 0)
+			(end 2.25 0)
 			(stroke
 				(width 0.1)
@@
 		)
 		(fp_text user "${REFERENCE}"
-			(at 5.08 0 0)
+			(at 2.54 -3.37 90)
 			(layer "F.Fab")
 			(effects
@@
 		)
 		(pad "1" thru_hole circle
-			(at 0 0)
-			(size 1.6 1.6)
-			(drill 0.8)
+			(at 0 0 270)
+			(size 2.4 2.4)
+			(drill 1.2)
 			(layers "*.Cu" "*.Mask")
 			(remove_unused_layers no)
@@
 		)
 		(pad "2" thru_hole circle
-			(at 10.16 0)
-			(size 1.6 1.6)
-			(drill 0.8)
+			(at 5.08 0 270)
+			(size 2.4 2.4)
+			(drill 1.2)
 			(layers "*.Cu" "*.Mask")
 			(remove_unused_layers no)
@@
 		)
 		(embedded_fonts no)
-		(model "${KICAD10_3DMODEL_DIR}/Resistor_THT.3dshapes/R_Axial_DIN0207_L6.3mm_D2.5mm_P10.16mm_Horizontal.step"
+		(model "${KICAD10_3DMODEL_DIR}/Resistor_THT.3dshapes/R_Axial_DIN0414_L11.9mm_D4.5mm_P5.08mm_Vertical.step"
 			(offset
 				(xyz 0 0 0)
@@
 	(footprint "Capacitor_THT:CP_Radial_D4.0mm_P2.00mm"
 		(layer "F.Cu")
-		(at 128.25 118)
+		(at 131.127401 115.35)
 		(descr "CP, Radial series, Radial, pin pitch=2.00mm, diameter=4mm, height=7mm, Electrolytic Capacitor")
 		(tags "CP Radial series Radial pin pitch 2.00mm diameter 4mm height 7mm Electrolytic Capacitor")
@@
 		(polygon
 			(pts
-				(xy 138.25 126.5) (xy 138.25 120) (xy 129.25 120) (xy 129.25 108) (xy 125.25 108) (xy 125.25 112)
+				(xy 138.25 126.5) (xy 138.25 120) (xy 132.3 120) (xy 132.3 108) (xy 125.25 108) (xy 125.25 112)
 				(xy 124.5 112.75) (xy 122.25 112.75) (xy 122.25 121) (xy 124.75 121) (xy 125.25 121.5) (xy 125.25 126.5)
 			)
@@
 		(polygon
 			(pts
-				(xy 138.25 126.5) (xy 141.25 126.5) (xy 141.25 107.75) (xy 132 107.75) (xy 132 92.75) (xy 128.75 92.75)
-				(xy 128.75 106) (xy 127.75 107) (xy 129.25 108.5) (xy 129.25 119.75) (xy 137 119.75) (xy 138.25 121)
+				(xy 138.2 126.5) (xy 141.2 126.5) (xy 141.2 107.75) (xy 131.95 107.75) (xy 131.95 92.75) (xy 128.7 92.75)
+				(xy 128.7 106) (xy 127.7 107) (xy 129.2 108.5) (xy 129.231237 113.294896) (xy 131.2 113.3) (xy 132 114.1)
+				(xy 132 119.7) (xy 136.95 119.75) (xy 138.2 121)
 			)
 		)
