File: designs/sepic/pcb/sepic/sepic.kicad_sch (KiCad schematic)
At the start: 0 parts

Commit message: ss
Parts:
- added Co1, Cs1: 4.7u, Capacitor_THT:CP_Radial_D4.0mm_P2.00mm, symbol Device:C_Polarized
- added Co2, Cs2: 1u, Capacitor_THT:CP_Radial_D4.0mm_P2.00mm, symbol Device:C_Polarized
- added Co3: 10u, Capacitor_THT:CP_Radial_D4.0mm_P2.00mm, symbol Device:C_Polarized
- added Current_sensor1: 3.3v, Connector_PinSocket_2.54mm:PinSocket_1x02_P2.54mm_Vertical, symbol Connector:Conn_01x02_Socket
- added D1: D_Schottky, Diode_THT:D_DO-201AE_P15.24mm_Horizontal, symbol Device:D_Schottky
- added J2: output, TerminalBlock_Phoenix:TerminalBlock_Phoenix_MKDS-1,5-2-5.08_1x02_P5.08mm_Horizontal, symbol Connector:Screw_Terminal_01x02
- added J3: pwm, TerminalBlock_Phoenix:TerminalBlock_Phoenix_MKDS-1,5-2-5.08_1x02_P5.08mm_Horizontal, symbol Connector:Screw_Terminal_01x02
- added L1: 300u, custom_footprints:inductor_20x7.5, symbol Device:L
- added L2: 500u, custom_footprints:inductor_20x7.5, symbol Device:L
- added Q1: irfz44n, Package_TO_SOT_THT:TO-220-3_Vertical, symbol custom:irfz44n
- added R_c1, R_c2: 50m, Resistor_THT:R_Axial_DIN0207_L6.3mm_D2.5mm_P10.16mm_Horizontal, symbol Device:R
- added R_g1: 10m, Resistor_THT:R_Axial_DIN0207_L6.3mm_D2.5mm_P10.16mm_Horizontal, symbol Device:R
- added U1, U2: INA240A1D, Package_SO:SOIC-8_3.9x4.9mm_P1.27mm, symbol Amplifier_Current:INA240A1D
- added U3: TC4422, Package_DIP:DIP-8_W7.62mm, symbol Driver_FET:TC4422
- added Vcs1, iL1, iL2: Conn_01x02_Pin, Connector_PinHeader_2.54mm:PinHeader_1x02_P2.54mm_Vertical, symbol Connector:Conn_01x02_Pin
- added input1: input, TerminalBlock_Phoenix:TerminalBlock_Phoenix_MKDS-1,5-2-5.08_1x02_P5.08mm_Horizontal, symbol Connector:Screw_Terminal_01x02
Connections:
- new net: U1.5, iL1.2 (Pin_2)
- new net: Cs1.2, Cs2.2, D1.2 (A), L2.1, Vcs1.1 (Pin_1)
- new net: Current_sensor1.2 (Pin_2), U1.3 (REF2), U1.6 (V+), U2.3 (REF2), U2.6 (V+)
- new net: U2.5, iL2.2 (Pin_2)
- new net: L1.1, U3.1 (VDD), U3.8 (VDD), input1.2 (Pin_2)
- new net: Q1.1 (G), R_g1.2
- new net: J3.2 (Pin_2), U3.2 (INPUT)
- new net GND: Co1.2, Co2.2, Co3.2, Current_sensor1.1 (Pin_1), J2.2 (Pin_2), J3.1 (Pin_1), Q1.3 (S), R_c2.1, U1.2 (GND), U1.4 (GND), U1.7 (REF1), U2.1 (-), U2.2 (GND), U2.4 (GND), U2.7 (REF1), U3.4 (GND), U3.5 (GND), iL1.1 (Pin_1), iL2.1 (Pin_1), input1.1 (Pin_1)
- new net R_c2n: L2.2, R_c2.2, U2.8 (+)
- new net R_cn: Cs1.1, Cs2.1, Q1.2 (D), R_c1.2, U1.1 (-), Vcs1.2 (Pin_2)
- new net R_cp: L1.2, R_c1.1, U1.8 (+)
- new net Vo: Co1.1, Co2.1, Co3.1, D1.1 (K), J2.1 (Pin_1)
- new net pwm: R_g1.1, U3.6 (OUTPUT), U3.7 (OUTPUT)
Other:
- note added: "TODO: Check mosfet pinout,50M RESISTOR FOOTPRINT check inductors footprint"

Commit message: pcb
Parts:
- added C1: 2.2u, Capacitor_THT:C_Disc_D5.0mm_W2.5mm_P2.50mm, symbol Device:C
- R_g1: value 10m -> 10
Connections:
- net GND: now also C1.2
- net at L1.1, U3.1 (VDD), U3.8 (VDD)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: now also C1.1
Other:
- note removed: "TODO: Check mosfet pinout,50M RESISTOR FOOTPRINT check inductors footprint"
Changed lines of the file:
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@@
 	(generator_version "10.0")
 	(paper "A4")
-	(text "TODO: Check mosfet pinout,50M RESISTOR FOOTPRINT\ncheck inductors footprint\n"
-		(exclude_from_sim no)
-		(at 164.846 55.88 0)
-		(effects
-			(font
-				(size 1.27 1.27)
-			)
-		)
-	)
 	(junction
 		(at 190.5 88.9)
@@
 	)
 	(junction
+		(at 88.9 114.3)
+		(diameter 0)
+		(color 0 0 0 0)
+	)
+	(junction
 		(at 144.78 78.74)
 		(diameter 0)
@@
 	)
 	(junction
+		(at 88.9 88.9)
+		(diameter 0)
+		(color 0 0 0 0)
+	)
+	(junction
 		(at 137.16 78.74)
 		(diameter 0)
@@
 	(wire
 		(pts
-			(xy 81.28 88.9) (xy 93.98 88.9)
+			(xy 81.28 88.9) (xy 88.9 88.9)
 		)
 		(stroke
@@
 	(wire
 		(pts
+			(xy 88.9 88.9) (xy 93.98 88.9)
+		)
+		(stroke
+			(width 0)
+			(type default)
+		)
+	)
+	(wire
+		(pts
 			(xy 139.7 63.5) (xy 134.62 63.5)
 		)
@@
 	(wire
 		(pts
+			(xy 88.9 105.41) (xy 88.9 114.3)
+		)
+		(stroke
+			(width 0)
+			(type default)
+		)
+	)
+	(wire
+		(pts
 			(xy 105.41 46.99) (xy 105.41 55.88)
 		)
@@
 	(wire
 		(pts
+			(xy 88.9 88.9) (xy 88.9 97.79)
+		)
+		(stroke
+			(width 0)
+			(type default)
+		)
+	)
+	(wire
+		(pts
 			(xy 172.72 114.3) (xy 172.72 104.14)
 		)
@@
 	(wire
 		(pts
-			(xy 81.28 114.3) (xy 114.3 114.3)
+			(xy 88.9 114.3) (xy 114.3 114.3)
+		)
+		(stroke
+			(width 0)
+			(type default)
+		)
+	)
+	(wire
+		(pts
+			(xy 81.28 114.3) (xy 88.9 114.3)
 		)
 		(stroke
@@
 	)
 	(symbol
+		(lib_id "Device:C")
+		(at 88.9 101.6 0)
+		(unit 1)
+		(body_style 1)
+		(exclude_from_sim no)
+		(in_bom yes)
+		(on_board yes)
+		(in_pos_files yes)
+		(dnp no)
+		(property "Reference" "C1"
+			(at 85.09 99.06 0)
+			(show_name no)
+			(do_not_autoplace no)
+			(effects
+				(font
+					(size 1.27 1.27)
+				)
+				(justify left)
+			)
+		)
+		(property "Value" "2.2u"
+			(at 86.36 104.648 0)
+			(show_name no)
+			(do_not_autoplace no)
+			(effects
+				(font
+					(size 1.27 1.27)
+				)
+				(justify left)
+			)
+		)
+		(property "Footprint" "Capacitor_THT:C_Disc_D5.0mm_W2.5mm_P2.50mm"
+			(at 89.8652 105.41 0)
+			(hide yes)
+			(show_name no)
+			(do_not_autoplace no)
+			(effects
+				(font
+					(size 1.27 1.27)
+				)
+			)
+		)
+		(property "Datasheet" ""
+			(at 88.9 101.6 0)
+			(hide yes)
+			(show_name no)
+			(do_not_autoplace no)
+			(effects
+				(font
+					(size 1.27 1.27)
+				)
+			)
+		)
+		(property "Description" "Unpolarized capacitor"
+			(at 88.9 101.6 0)
+			(hide yes)
+			(show_name no)
+			(do_not_autoplace no)
+			(effects
+				(font
+					(size 1.27 1.27)
+				)
+			)
+		)
+		(pin "2"
+		)
+		(pin "1"
+		)
+		(instances
+			(project "sepic"
+				(path "/90bfeea5-c5c2-4088-b876-270f7583e2b4"
+					(reference "C1")
+					(unit 1)
+				)
+			)
+		)
+	)
+	(symbol
 		(lib_id "Device:R")
 		(at 154.94 105.41 180)
@@
 			)
 		)
-		(property "Value" "10m"
+		(property "Value" "10"
 			(at 115.57 95.25 90)
 			(show_name no)

Commit message: test
Parts:
- added H1, H2, H3, H4: MountingHole, MountingHole:MountingHole_3.2mm_M3_DIN965, symbol Mechanical:MountingHole

Commit message: update
Parts:
- R_c1: footprint Resistor_THT:R_Axial_DIN0207_L6.3mm_D2.5mm_P10.16mm_Horizontal -> Resistor_THT:R_Axial_DIN0414_L11.9mm_D4.5mm_P15.24mm_Horizontal
- R_c2: footprint Resistor_THT:R_Axial_DIN0207_L6.3mm_D2.5mm_P10.16mm_Horizontal -> Resistor_THT:R_Axial_DIN0414_L11.9mm_D4.5mm_P5.08mm_Vertical
Changed lines of the file:
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@@
 			)
 		)
-		(property "Footprint" "Resistor_THT:R_Axial_DIN0207_L6.3mm_D2.5mm_P10.16mm_Horizontal"
+		(property "Footprint" "Resistor_THT:R_Axial_DIN0414_L11.9mm_D4.5mm_P5.08mm_Vertical"
 			(at 156.718 105.41 90)
 			(hide yes)
@@
 			)
 		)
-		(property "Footprint" "Resistor_THT:R_Axial_DIN0207_L6.3mm_D2.5mm_P10.16mm_Horizontal"
+		(property "Footprint" "Resistor_THT:R_Axial_DIN0414_L11.9mm_D4.5mm_P15.24mm_Horizontal"
 			(at 114.3 90.678 90)
 			(hide yes)
